Commit message: removed trailing spaces that were breaking *.launch.*

File: urdf/snake_robot_core.xacro (robot description, xacro)
@@ -35,5 +35,5 @@
         <parent link="link_1"/>
         <child link="link_2"/>
-        <limit lower="-0.785398163397 " upper="0.785398163397" velocity="50.0" effort="1000.0"/>
+        <limit lower="-0.785398163397" upper="0.785398163397" velocity="50.0" effort="1000.0"/>
         <origin xyz="0.0 0.175 0.0" rpy="0 0 0"/>
         <axis xyz="0 0 1"/>
@@ -63,5 +63,5 @@
         <parent link="link_2"/>
         <child link="link_3"/>
-        <limit lower="-0.785398163397 " upper="0.785398163397" velocity="50.0" effort="1000.0"/>
+        <limit lower="-0.785398163397" upper="0.785398163397" velocity="50.0" effort="1000.0"/>
         <origin xyz="0.0 0.175 0.0" rpy="0 0 0"/>
         <axis xyz="0 0 1"/>
@@ -91,5 +91,5 @@
         <parent link="link_3"/>
         <child link="link_4"/>
-        <limit lower="-0.785398163397 " upper="0.785398163397" velocity="50.0" effort="1000.0"/>
+        <limit lower="-0.785398163397" upper="0.785398163397" velocity="50.0" effort="1000.0"/>
         <origin xyz="0.0 0.175 0.0" rpy="0 0 0"/>
         <axis xyz="0 0 1"/>
@@ -118,5 +118,5 @@
         <parent link="link_4"/>
         <child link="link_5"/>
-        <limit lower="-0.785398163397 " upper="0.785398163397" velocity="50.0" effort="1000.0"/>
+        <limit lower="-0.785398163397" upper="0.785398163397" velocity="50.0" effort="1000.0"/>
         <origin xyz="0.0 0.175 0.0" rpy="0 0 0"/>
         <axis xyz="0 0 1"/>
@@ -145,5 +145,5 @@
         <parent link="link_5"/>
         <child link="link_6"/>
-        <limit lower="-0.785398163397 " upper="0.785398163397" velocity="50.0" effort="1000.0"/>
+        <limit lower="-0.785398163397" upper="0.785398163397" velocity="50.0" effort="1000.0"/>
         <origin xyz="0.0 0.175 0.0" rpy="0 0 0"/>
         <axis xyz="0 0 1"/>
@@ -173,5 +173,5 @@
         <parent link="link_6"/>
         <child link="link_7"/>
-        <limit lower="-0.785398163397 " upper="0.785398163397" velocity="50.0" effort="1000.0"/>
+        <limit lower="-0.785398163397" upper="0.785398163397" velocity="50.0" effort="1000.0"/>
         <origin xyz="0.0 0.175 0.0" rpy="0 0 0"/>
         <axis xyz="0 0 1"/>
@@ -201,5 +201,5 @@
         <parent link="link_7"/>
         <child link="link_8"/>
-        <limit lower="-0.785398163397 " upper="0.785398163397" velocity="50.0" effort="1000.0"/>
+        <limit lower="-0.785398163397" upper="0.785398163397" velocity="50.0" effort="1000.0"/>
         <origin xyz="0.0 0.175 0.0" rpy="0 0 0"/>
         <axis xyz="0 0 1"/>
@@ -229,5 +229,5 @@
         <parent link="link_8"/>
         <child link="link_9"/>
-        <limit lower="-0.785398163397 " upper="0.785398163397" velocity="50.0" effort="1000.0"/>
+        <limit lower="-0.785398163397" upper="0.785398163397" velocity="50.0" effort="1000.0"/>
         <origin xyz="0.0 0.175 0.0" rpy="0 0 0"/>
         <axis xyz="0 0 1"/>
@@ -257,5 +257,5 @@
         <parent link="link_9"/>
         <child link="link_10"/>
-        <limit lower="-0.785398163397 " upper="0.785398163397" velocity="50.0" effort="1000.0"/>
+        <limit lower="-0.785398163397" upper="0.785398163397" velocity="50.0" effort="1000.0"/>
         <origin xyz="0.0 0.175 0.0" rpy="0 0 0"/>
         <axis xyz="0 0 1"/>
